File: ThunderHorse.kicad_pcb (KiCad board)
At the start: 6 copper layers, 112.5 x 60 mm, 252 parts, among them J1 JTAG, J10 MOTOR2, J11 SWD3, J12 MOTOR3, J13 SWD4, J14 MOTOR4, J16 UFL, J2 HH-16P-CB-TYPE-C, J3 GPS, J4 CAM, J5 GPS, J6 CAM, J7 SWD1, J8 MOTOR1, J9 SWD2, Q1 SI2301BDS, Q10 XRS306D, Q11 XRS306D, Q12 XRS306D, Q13 XRS306D, Q14 SI2312BDS, Q2 XRS306D, Q3 XRS306D, Q4 XRS306D, Q5 XRS306D, Q6 XRS306D, Q7 XRS306D, Q8 XRS306D, Q9 XRS306D, SW1 TS2306A, SW2 TS2306A, U1 21700_DUAL_HOLDER, U10 DRV8300D, U11 STM32G071GBUxN, U12 DRV8300D, U13 STM32G071GBUxN, U14 DRV8300D, U15 TPRT9013-33, U16 ICM-42688-P, U17 BMP280, U18 INA230, U19 TPRT9013-33, U2 TPS63070RNMR, U20 SX1280IMLTRT, U21 AT2401C, U3 TPRT9013-33, U4 RP2354B, U5 W25Q128JVPIQ, U6 USBLC6-2P6, U7 STM32G071GBUxN, U8 DRV8300D, U9 STM32G071GBUxN, Y1 40MHz, Y2 52MHz/10ppm

Commit message: ESC layout and footprints
Added the initial ESC layout.
Updated some footprints for compatibility.
Parts:
- removed the C46 at (202.3, 18.5)
- removed the Q2 at (186.7, 37.5)
- added C42: 10u, Capacitor_SMD:C_1206_3216Metric, F.Cu at (119.8, 79.8)
- added C79: 10u, Capacitor_SMD:C_0805_2012Metric, F.Cu at (163.3, 158.9)
- added C80: 1u, Capacitor_SMD:C_0603_1608Metric, F.Cu at (151.0, 151.1)
- added C81: 1u, Capacitor_SMD:C_0603_1608Metric, F.Cu at (151.0, 153.6)
- added C82: 1u, Capacitor_SMD:C_0603_1608Metric, F.Cu at (151.0, 156.1)
- added Q2: XRS306D, Custom_Parts:PDFN8_DUAL_3.3x3.3mm, F.Cu at (1.82, 3.02)
- added Q2: XRS306D, Custom_Parts:PDFN8_DUAL_3.3x3.3mm, F.Cu at (135.1, 77.5)
- C11, C3: footprint Capacitor_SMD:C_0805_2012Metric -> Capacitor_SMD:C_0603_1608Metric
- C47, C58, C69, C71: value 10u -> 1u; footprint Capacitor_SMD:C_1206_3216Metric -> Capacitor_SMD:C_0603_1608Metric
- C48: value 100n -> 10u; footprint Capacitor_SMD:C_0603_1608Metric -> Capacitor_SMD:C_1206_3216Metric
- C49, C61, C73: value 10u -> 100n; footprint Capacitor_SMD:C_1206_3216Metric -> Capacitor_SMD:C_0603_1608Metric
- C53, C64, C75: footprint Capacitor_SMD:C_0805_2012Metric -> Capacitor_SMD:C_1206_3216Metric
- C54, C65, C66, C76, C77, C78: value 1u -> 10u; footprint Capacitor_SMD:C_0603_1608Metric -> Capacitor_SMD:C_1206_3216Metric
- C55, C67: value 1u -> 10u; footprint Capacitor_SMD:C_0603_1608Metric -> Capacitor_SMD:C_0805_2012Metric
- C59, C70: value 100n -> 1u
- J10, J12, J14, J8: footprint Custom_Parts:PAD_3_SQUARE_SOLID_2.0x2.0mm_P2.5mm -> Custom_Parts:PAD_3_SQUARE_SOLID_2.5x2.5mm_P4.0mm; moved to B.Cu
- J3, J4: moved to B.Cu
- U20: footprint Package_DFN_QFN:QFN-24-1EP_4x4mm_P0.5mm_EP2.6x2.6mm_ThermalVias -> Custom_Parts:QFN-24_4x4mm_P0.5mm_EP
- U21: footprint Package_DFN_QFN:QFN-16-1EP_3x3mm_P0.5mm_EP1.7x1.7mm_ThermalVias -> Custom_Parts:QFN-16_3x3mm_P0.5mm_EP1.7x1.7mm_EP
- moved C64 212.5 mm to (104.6, 157.0)
- moved C60 207.9 mm to (104.6, 147.0)
- moved C66 206.3 mm to (104.6, 163.7)
- moved Q10 206.0 mm to (119.0, 166.4)
- moved Q8 206.0 mm to (109.7, 166.4)
- moved Q9 206.0 mm to (114.4, 166.4)
- moved C62 205.9 mm to (104.6, 150.3)
- moved C63 205.9 mm to (104.6, 153.7)
- moved C65 205.7 mm to (104.6, 160.4)
- moved C61 203.3 mm to (109.4, 149.1)
- moved U11 200.6 mm to (123.0, 148.5)
- moved U12 200.6 mm to (122.6, 154.8)
- moved R51 196.3 mm to (109.4, 159.1)
- moved R52 196.3 mm to (109.4, 161.6)
- moved R53 196.3 mm to (113.4, 146.6)
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- renumbered C96 to C100, C100 to C104, C101 to C105, C42 to C43, C43 to C44, C44 to C45, C45 to C46, C79 to C83, C80 to C84, C81 to C85, C82 to C86, C83 to C87, C84 to C88, C85 to C89, C86 to C90, C87 to C91, C88 to C92, C89 to C93, C90 to C94, C91 to C95, C92 to C96, C94 to C98
Connections:
- C47 pad 1: VBAT -> 3V3
- C48 pad 1: 3V3 -> VBAT
- C49 pad 1: VBAT -> 3V3
- C53 pad 1: 5V -> VBAT
- C54 pad 1: /ESC/ESC2/BSTA -> VBAT
- C54 pad 2: /ESC/ESC2/MOTOR_A -> GND
- C55 pad 1: /ESC/ESC2/BSTB -> 5V
- C55 pad 2: /ESC/ESC2/MOTOR_B -> GND
- C56 pad 1: /ESC/ESC2/BSTC -> /ESC/ESC2/BSTA
- C56 pad 2: /ESC/ESC2/MOTOR_C -> /ESC/ESC2/MOTOR_A
- C57 pad 1: 3V3 -> /ESC/ESC2/BSTB
- C57 pad 2: GND -> /ESC/ESC2/MOTOR_B
- C58 pad 1: VBAT -> /ESC/ESC2/BSTC
- C58 pad 2: GND -> /ESC/ESC2/MOTOR_C
- C61 pad 1: VBAT -> 3V3
- C64 pad 1: 5V -> VBAT
- C65 pad 1: /ESC/ESC3/BSTA -> VBAT
- C65 pad 2: /ESC/ESC3/MOTOR_A -> GND
- C66 pad 1: /ESC/ESC3/BSTB -> VBAT
- C66 pad 2: /ESC/ESC3/MOTOR_B -> GND
- C67 pad 1: /ESC/ESC3/BSTC -> 5V
- C67 pad 2: /ESC/ESC3/MOTOR_C -> GND
- C68 pad 1: 3V3 -> /ESC/ESC3/BSTA
- C68 pad 2: GND -> /ESC/ESC3/MOTOR_A
- C69 pad 1: VBAT -> /ESC/ESC3/BSTB
- C69 pad 2: GND -> /ESC/ESC3/MOTOR_B
- C70 pad 1: 3V3 -> /ESC/ESC3/BSTC
- C70 pad 2: GND -> /ESC/ESC3/MOTOR_C
- C71 pad 1: VBAT -> 3V3
- C73 pad 1: VBAT -> 3V3
- C75 pad 1: 5V -> VBAT
- C76 pad 1: /ESC/ESC4/BSTA -> VBAT
- C76 pad 2: /ESC/ESC4/MOTOR_A -> GND
- C77 pad 1: /ESC/ESC4/BSTB -> VBAT
- C77 pad 2: /ESC/ESC4/MOTOR_B -> GND
- C78 pad 1: /ESC/ESC4/BSTC -> VBAT
- C78 pad 2: /ESC/ESC4/MOTOR_C -> GND
Other:
- board size 112.5 x 60 mm -> 105.8 x 60 mm

Commit message: Layout replication
Updated the ESC schematic to allow for layout replication.
Updated the PCB layout.
Parts:
- removed the Q2 at (1.82, 3.02)
- J10: value MOTOR2 -> MOTOR1
- J11: value SWD3 -> SWD1
- J12: value MOTOR3 -> MOTOR1
- J13: value SWD4 -> SWD1
- J14: value MOTOR4 -> MOTOR1
- J9: value SWD2 -> SWD1
- moved BZ1 159.1 mm to (98.6, 100.0), turned to 90 degrees
- moved J6 146.7 mm to (96.8, 116.4), turned to -90 degrees
- moved J4 135.2 mm to (103.4, 124.6)
- moved J16 94.1 mm to (96.7, 91.8), turned to 180 degrees
- moved C96 94.1 mm to (96.7, 79.2), turned to 180 degrees
- moved L3 93.7 mm to (96.7, 80.8), turned to 180 degrees
- moved C95 93.4 mm to (96.7, 82.3), turned to 180 degrees
- moved R87 93.3 mm to (96.7, 86.5), turned to 180 degrees
- moved R86 93.3 mm to (96.7, 85.0), turned to 180 degrees
- moved C94 88.3 mm to (99.9, 77.3), turned to 180 degrees
- moved FL1 86.6 mm to (100.5, 91.8), turned to -90 degrees
- moved U20 84.1 mm to (101.5, 81.5), turned to 180 degrees
- moved U21 84.0 mm to (101.4, 87.6), turned to -90 degrees
- moved C90 79.6 mm to (104.5, 94.2), turned to 180 degrees
- moved C93 78.8 mm to (104.5, 92.0), turned to 180 degrees
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Other:
- board size 105.8 x 60 mm -> 99.1 x 60 mm

Commit message: Initial layout
Completed an initial layout of the main components.

TODO
Route the ESCs and check the result.
Parts:
- removed the D1 at (172.9, 106.6)
- removed the Q1 at (172.9, 109.8)
- removed the R18 at (175.6, 107.6)
- added C16: 100n, Capacitor_SMD:C_0603_1608Metric, F.Cu at (164.4, 103.5)
- added J17: IO1, Custom_Parts:PAD_6_SQUARE_SOLID_1.5x1.5mm_P2.0mm, B.Cu at (176.6, 124.6)
- added J18: IO2, Custom_Parts:PAD_6_SQUARE_SOLID_1.5x1.5mm_P2.0mm, B.Cu at (103.4, 75.4)
- added R5: 33K, Resistor_SMD:R_0603_1608Metric, F.Cu at (167.6, 103.5)
- added U4: TPS2121, Custom_Parts:VQFN-HR-12_2x2.5mm_P0.5mm, F.Cu at (166.1, 106.2)
- C19: renamed from C18; footprint Capacitor_SMD:C_0805_2012Metric -> Capacitor_SMD:C_0603_1608Metric
- C27: renamed from C26; footprint Capacitor_SMD:C_0805_2012Metric -> Capacitor_SMD:C_0603_1608Metric
- C31: renamed from C30; footprint Capacitor_SMD:C_0805_2012Metric -> Capacitor_SMD:C_0603_1608Metric
- C34: renamed from C33; footprint Capacitor_SMD:C_0805_2012Metric -> Capacitor_SMD:C_0603_1608Metric
- C90: renamed from C89; footprint Capacitor_SMD:C_0201_0603Metric -> Capacitor_SMD:C_0603_1608Metric
- U1: value 21700_DUAL_HOLDER -> BATTERY
- moved Q13 187.1 mm to (96.8, 107.8), turned to 180 degrees
- moved R89 174.0 mm to (99.0, 110.4), turned to 180 degrees
- moved R90 171.5 mm to (100.0, 107.8), turned to 90 degrees
- moved C34 142.7 mm to (131.4, 99.8), turned to 180 degrees
- moved L2 135.9 mm to (150.6, 104.4), turned to -90 degrees
- moved Y1 135.7 mm to (130.4, 104.2), turned to 180 degrees
- moved C27 135.0 mm to (145.0, 108.2), turned to -90 degrees
- moved R13 134.3 mm to (132.8, 105.7), turned to 90 degrees
- moved C26 133.6 mm to (131.4, 98.2), turned to 180 degrees
- moved C17 132.3 mm to (130.4, 102.0), turned to 180 degrees
- moved C28 132.2 mm to (136.2, 108.2), turned to -90 degrees
- moved C19 131.4 mm to (148.6, 104.4), turned to -90 degrees
- moved C21 131.1 mm to (130.4, 106.4)
- moved C31 130.5 mm to (147.0, 104.4), turned to -90 degrees
- moved C29 128.6 mm to (139.0, 108.2), turned to -90 degrees
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- renumbered C100 to C101, C104 to C105, C105 to C106, C16 to C17, C17 to C18, C19 to C20, C20 to C21, C21 to C22, C22 to C23, C23 to C24, C24 to C25, C25 to C26, C27 to C28, C28 to C29, C29 to C30, C31 to C32, C32 to C33, C34 to C35, C35 to C36, C36 to C37, C37 to C38, C38 to C39, C39 to C40, C40 to C41, C41 to C42, C42 to C43, C43 to C44, C44 to C45, C45 to C46, C46 to C47, C47 to C48, C48 to C49, C49 to C50, C50 to C51, C51 to C52, C52 to C53, C53 to C54, C54 to C55, C55 to C56, C56 to C57, C57 to C58, C58 to C59, C59 to C60, C60 to C61, C61 to C62, C62 to C63, C63 to C64, C64 to C65, C65 to C66, C66 to C67, C67 to C68, C68 to C69, C69 to C70, C70 to C71, C71 to C72, C72 to C73, C73 to C74, C74 to C75, C75 to C76, C76 to C77, C77 to C78, C78 to C79, C79 to C80, C80 to C81, C81 to C82, C82 to C83, C83 to C84, C84 to C85, C85 to C86, C86 to C87, C87 to C88, C88 to C89, C90 to C91, C91 to C92, C92 to C93, C93 to C94, C94 to C95, C95 to C96, C96 to C97, C98 to C99, D2 to D1, D3 to D2, Q2 to Q1, Q11 to Q10, Q12 to Q11, Q13 to Q12, Q14 to Q13, Q3 to Q2, Q4 to Q3, Q5 to Q4, Q6 to Q5, Q7 to Q6, Q8 to Q7, Q9 to Q8, Q10 to Q9, R9 to R10, R10 to R11, R11 to R12, R12 to R13, R13 to R14, R14 to R15, R15 to R16, R16 to R17, R17 to R18, R5 to R6, R6 to R7, R7 to R8, R8 to R9, U9 to U10, U10 to U11, U11 to U12, U12 to U13, U13 to U14, U14 to U15, U15 to U16, U16 to U17, U17 to U18, U18 to U19, U19 to U20, U20 to U21, U21 to U22, U4 to U5, U5 to U6, U6 to U7, U7 to U8, U8 to U9
Connections:
- net /MCU/VBUS renamed VBUS
- BZ1 pad 1: 5V -> 5V_REG
- U18 pad 2: 3V3_IMU -> 3V3
- U18 pad 5: 3V3_IMU -> 3V3
- U5 pad 47: unconnected-(U4-GPIO38-Pad47) -> GPIO38
- U5 pad 48: unconnected-(U4-GPIO39-Pad48) -> GPIO39
- U5 pad 57: unconnected-(U4-GPIO46/ADC6-Pad57) -> GPIO46
- U5 pad 58: unconnected-(U4-GPIO47/ADC7-Pad58) -> GPIO47
- U5 pad 6: unconnected-(U4-GPIO8-Pad6) -> GPIO8
- U5 pad 7: unconnected-(U4-GPIO9-Pad7) -> GPIO9
- U5 pad 79: unconnected-(U4-GPIO2-Pad79) -> GPIO2
- U5 pad 80: unconnected-(U4-GPIO3-Pad80) -> GPIO3
Routing:
- net VBAT: track 0.00 -> 4.27 mm, vias 0 -> 18
- net VBAT_IN: track 0.00 -> 3.54 mm, vias 0 -> 18
- net GND: track 0.00 -> 2.05 mm, vias 0 -> 18
- net 3V3: track 0.00 -> 1.94 mm
- added copper zone on F.Cu, net VBAT
- added copper zone on F.Cu, net VBAT_IN
