File: ESC1.kicad_sch (KiCad schematic)
At the start: 35 parts, among them J1 MOTOR_A, J4 MOTOR_B, J5 MOTOR_C, Q1 Q_NMOS_GDS, Q2 Q_NMOS_GDS, Q3 Q_NMOS_GDS, Q4 Q_NMOS_GDS, Q5 Q_NMOS_GDS, Q6 Q_NMOS_GDS, U5 STM32G071GBUxN, U6 DRV8300D

Commit message: Footprints and revision
Added the missing footprints.
Updated a all the schematics.
Completed an initial review of the schematics.

TODO:
Perform a deep review of the schematics before committing to layout.
Parts:
- removed Q1, Q2, Q3, Q4, Q5, Q6: Q_NMOS_GDS, symbol Transistor_FET:Q_NMOS_GDS
- added Q3, Q4, Q5: XRS306D, Custom_Parts:PDFN8, symbol Transistor_FET:Q_Dual_NMOS_S1G1S2G2D2D1
- C63: renamed from C40; footprint (none) -> Capacitor_SMD:C_0603_1608Metric
- C64: renamed from C39; footprint (none) -> Capacitor_SMD:C_0603_1608Metric
- C65: renamed from C38; footprint (none) -> Capacitor_SMD:C_0805_2012Metric
- C66: renamed from C35; footprint (none) -> Capacitor_SMD:C_0603_1608Metric
- C67: renamed from C36; footprint (none) -> Capacitor_SMD:C_0603_1608Metric
- C68: renamed from C37; footprint (none) -> Capacitor_SMD:C_0603_1608Metric
- R28: renamed from R16; footprint (none) -> Resistor_SMD:R_0603_1608Metric
- R29: renamed from R17; footprint (none) -> Resistor_SMD:R_0603_1608Metric
- R30: renamed from R18; footprint (none) -> Resistor_SMD:R_0603_1608Metric
- R31: renamed from R15; footprint (none) -> Resistor_SMD:R_0603_1608Metric
- R32: renamed from R19; footprint (none) -> Resistor_SMD:R_0603_1608Metric
- R33: renamed from R20; footprint (none) -> Resistor_SMD:R_0603_1608Metric
- R34: renamed from R21; footprint (none) -> Resistor_SMD:R_0603_1608Metric
- R35: renamed from R22; footprint (none) -> Resistor_SMD:R_0603_1608Metric
- R36: renamed from R23; footprint (none) -> Resistor_SMD:R_0603_1608Metric
- R37: renamed from R24; footprint (none) -> Resistor_SMD:R_0603_1608Metric
- R38: renamed from R6; footprint (none) -> Resistor_SMD:R_0603_1608Metric
- R39: renamed from R7; footprint (none) -> Resistor_SMD:R_0603_1608Metric
- R40: renamed from R8; footprint (none) -> Resistor_SMD:R_0603_1608Metric
- R41: renamed from R9; footprint (none) -> Resistor_SMD:R_0603_1608Metric
- R42: renamed from R10; footprint (none) -> Resistor_SMD:R_0603_1608Metric
- R43: renamed from R11; footprint (none) -> Resistor_SMD:R_0603_1608Metric
- renumbered J1 to J5, J4 to J6, J5 to J7, TP1 to TP11, TP2 to TP12, U5 to U15, U6 to U16
Connections:
- net GND: now also Q3.3 (S), Q4.3 (S), Q5.3 (S)
- net MOTOR_A: now also Q3.1 (S), Q3.5 (D)
- net MOTOR_B: now also Q4.1 (S), Q4.5 (D)
- net MOTOR_C: now also Q5.1 (S), Q5.5 (D)
- net VBAT: now also Q3.6 (D), Q4.6 (D), Q5.6 (D)
- net at R40.2: now also Q4.2 (G)
- net at R41.2: now also Q4.4 (G)
- net at R42.2: now also Q5.2 (G)
- net at R43.2: now also Q5.4 (G)
- net at R39.2: now also Q3.4 (G)
- net at R38.2: now also Q3.2 (G)

Commit message: ESC design
Updated the ESC schematics.
Parts:
- renumbered C63 to C30, C64 to C31, C65 to C32, C66 to C33, C67 to C34, C68 to C35, J5 to J3, J6 to J4, J7 to J5, Q3 to Q2, Q4 to Q3, Q5 to Q4, R28 to R20, R29 to R21, R30 to R22, R31 to R23, R32 to R24, R33 to R25, R34 to R26, R35 to R27, R36 to R28, R37 to R29, R38 to R30, R39 to R31, R40 to R32, R41 to R33, R42 to R34, R43 to R35, U15 to U7, U16 to U8
Connections:
- net BSTB: now reaches C34.1, U8.17 (BSTB)
- net GHB_IN: now reaches Q3.2 (G), R32.2
- net GHC_IN: now reaches Q4.2 (G), R34.2
- net BSTC: now reaches C35.1, U8.14 (BSTC)
- net GLB_IN: now reaches Q3.4 (G), R33.2
- net BSTA: now reaches C33.1, U8.20 (BSTA)
- net GLC_IN: now reaches Q4.4 (G), R35.2
- net ESC: now reaches R23.1, U7.12 (PA6)
- net GLA_IN: now reaches Q2.4 (G), R31.2
- net GHA_IN: now reaches Q2.2 (G), R30.2
Other:
- company: (none) -> DavidMolTor
- title: (none) -> THUNDER HORSE
- moved on the sheet: J3, J4, J5, Q2A, Q2B, Q3A, Q3B, Q4A, Q4B

Commit message: Connectors and tag
Added bulk capacitance for each ESC.
Added SWD connector.
Updated all tags.

TODO:
Add pads for the unconnected GPIO pins.
Parts:
- removed J3: MOTOR_A, TestPoint:TestPoint_Pad_D2.0mm, symbol Connector:Conn_01x01_Socket
- removed J4: MOTOR_B, TestPoint:TestPoint_Pad_D2.0mm, symbol Connector:Conn_01x01_Socket
- removed J5: MOTOR_C, TestPoint:TestPoint_Pad_D2.0mm, symbol Connector:Conn_01x01_Socket
- removed TP11: SWDIO, TestPoint:TestPoint_Pad_D1.0mm, symbol Connector:TestPoint
- removed TP12: SWCLK, TestPoint:TestPoint_Pad_D1.0mm, symbol Connector:TestPoint
- added C36, C38, C39, C40, C41: 10u, symbol Device:C
- added J7: SWD1, symbol Connector_Generic:Conn_01x02
- added J8: MOTOR1, Custom_Parts:PAD_3_SQUARE_SOLID_2.0x2.0mm_P2.5mm, symbol Connector_Generic:Conn_01x03
- renumbered C30 to C35, C31 to C37, C32 to C42, C33 to C43, C34 to C44, C35 to C45, R20 to R19, R21 to R20, R22 to R21, R24 to R22, R25 to R24, R26 to R25, R27 to R26, R28 to R27, R29 to R28, R30 to R29, R31 to R30, R32 to R31, R33 to R32, R34 to R33, R35 to R34
Connections:
- net GND: now also C36.2, C38.2, C39.2, C40.2, C41.2
- net MOTOR_A: now also J8.1 (Pin_1)
- net MOTOR_B: now also J8.2 (Pin_2)
- net MOTOR_C: now also J8.3 (Pin_3)
- net SWCLK: now also J7.2 (Pin_2)
- net SWDIO: now also J7.1 (Pin_1)
- net VBAT: now also C36.1, C38.1, C39.1, C40.1, C41.1
Other:
- moved on the sheet: R19, R20, R21, R22, R24, R25, R26, R27, R28

Commit message: Missing labels and revision
First complete revision of the schematic.
Added missing labels.

TODO:
Continue reviewing the schematic.
Include net coloring.
Parts:
- C36, C38, C39, C40, C41: footprint (none) -> Capacitor_SMD:C_1206_3216Metric
- J7: footprint (none) -> Custom_Parts:PAD_2_SQUARE_SOLID_1.0x1.0mm_P1.5mm
- Q2, Q3, Q4: footprint Custom_Parts:PDFN8 -> Custom_Parts:PDFN8_DUAL_3.3x3.3mm
Connections:
- no-connect marks 13 -> 15
Changed lines of the file:
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@@
 	)
 	(no_connect
+		(at 143.51 81.28)
+	)
+	(no_connect
+		(at 143.51 83.82)
+	)
+	(no_connect
 		(at 50.8 54.61)
 	)
@@
 	(wire
 		(pts
-			(xy 140.97 81.28) (xy 140.97 97.79)
+			(xy 140.97 88.9) (xy 140.97 97.79)
 		)
 		(stroke
@@
 	(wire
 		(pts
-			(xy 143.51 81.28) (xy 140.97 81.28)
+			(xy 143.51 88.9) (xy 140.97 88.9)
 		)
 		(stroke
@@
 			)
 		)
-		(property "Footprint" ""
+		(property "Footprint" "Capacitor_SMD:C_1206_3216Metric"
 			(at 50.4952 180.34 0)
 			(effects
@@
 			)
 		)
-		(property "Footprint" "Custom_Parts:PDFN8"
+		(property "Footprint" "Custom_Parts:PDFN8_DUAL_3.3x3.3mm"
 			(at 248.92 125.73 0)
 			(effects
@@
 			)
 		)
-		(property "Footprint" "Custom_Parts:PDFN8"
+		(property "Footprint" "Custom_Parts:PDFN8_DUAL_3.3x3.3mm"
 			(at 248.92 82.55 0)
 			(effects
@@
 			)
 		)
-		(property "Footprint" ""
+		(property "Footprint" "Capacitor_SMD:C_1206_3216Metric"
 			(at 88.5952 180.34 0)
 			(effects
@@
 			)
 		)
-		(property "Footprint" "Custom_Parts:PDFN8"
+		(property "Footprint" "Custom_Parts:PDFN8_DUAL_3.3x3.3mm"
 			(at 248.92 95.25 0)
 			(effects
@@
 		(pin "4"
 		)
+		(pin "7"
+		)
+		(pin "8"
+		)
+		(pin "21"
+		)
+		(pin "5"
+		)
 		(instances
 			(project "ThunderHorse"
@@
 			)
 		)
-		(property "Footprint" ""
+		(property "Footprint" "Capacitor_SMD:C_1206_3216Metric"
 			(at 75.8952 180.34 0)
 			(effects
@@
 			)
 		)
-		(property "Footprint" "Custom_Parts:PDFN8"
+		(property "Footprint" "Custom_Parts:PDFN8_DUAL_3.3x3.3mm"
 			(at 248.92 52.07 0)
 			(effects
@@
 			)
 		)
-		(property "Footprint" ""
+		(property "Footprint" "Capacitor_SMD:C_1206_3216Metric"
 			(at 63.1952 180.34 0)
 			(effects
@@
 			)
 		)
-		(property "Footprint" ""
+		(property "Footprint" "Capacitor_SMD:C_1206_3216Metric"
 			(at 37.7952 180.34 0)
 			(effects
@@
 			)
 		)
-		(property "Footprint" "Custom_Parts:PDFN8"
+		(property "Footprint" "Custom_Parts:PDFN8_DUAL_3.3x3.3mm"
 			(at 248.92 138.43 0)
 			(effects
@@
 			)
 		)
-		(property "Footprint" ""
+		(property "Footprint" "Custom_Parts:PAD_2_SQUARE_SOLID_1.0x1.0mm_P1.5mm"
 			(at 102.87 77.47 0)
 			(effects
@@
 			)
 		)
-		(property "Footprint" "Custom_Parts:PDFN8"
+		(property "Footprint" "Custom_Parts:PDFN8_DUAL_3.3x3.3mm"
 			(at 248.92 39.37 0)
 			(effects

Commit message: ESC layout and footprints
Added the initial ESC layout.
Updated some footprints for compatibility.
Parts:
- added C42: 10u, Capacitor_SMD:C_1206_3216Metric, symbol Device:C
- J8: footprint Custom_Parts:PAD_3_SQUARE_SOLID_2.0x2.0mm_P2.5mm -> Custom_Parts:PAD_3_SQUARE_SOLID_2.5x2.5mm_P4.0mm
- renumbered C42 to C43, C43 to C44, C44 to C45, C45 to C46
Connections:
- net GND: now also C42.2
- net VBAT: now also C42.1
Changed lines of the file:
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@@
 		(exclude_from_sim no)
 		(at 22.86 161.29 0)
-		(size 80.01 29.21)
+		(size 93.98 29.21)
 		(margins 0.9525 0.9525 0.9525 0.9525)
 		(stroke
@@
 	)
 	(junction
+		(at 87.63 171.45)
+		(diameter 0)
+		(color 0 0 0 0)
+	)
+	(junction
 		(at 49.53 181.61)
 		(diameter 0)
@@
 	)
 	(junction
+		(at 68.58 171.45)
+		(diameter 0)
+		(color 0 0 0 0)
+	)
+	(junction
+		(at 87.63 181.61)
+		(diameter 0)
+		(color 0 0 0 0)
+	)
+	(junction
 		(at 41.91 39.37)
 		(diameter 0)
@@
 	)
 	(junction
+		(at 68.58 181.61)
+		(diameter 0)
+		(color 0 0 0 0)
+	)
+	(junction
 		(at 104.14 133.35)
 		(diameter 0)
@@
 	(wire
 		(pts
-			(xy 62.23 170.18) (xy 62.23 171.45)
+			(xy 68.58 170.18) (xy 68.58 171.45)
 		)
 		(stroke
@@
 	(wire
 		(pts
+			(xy 87.63 171.45) (xy 100.33 171.45)
+		)
+		(stroke
+			(width 0)
+			(type default)
+		)
+	)
+	(wire
+		(pts
+			(xy 87.63 181.61) (xy 100.33 181.61)
+		)
+		(stroke
+			(width 0)
+			(type default)
+		)
+	)
+	(wire
+		(pts
 			(xy 140.97 60.96) (xy 143.51 60.96)
 		)
@@
 	(wire
 		(pts
+			(xy 68.58 181.61) (xy 62.23 181.61)
+		)
+		(stroke
+			(width 0)
+			(type default)
+		)
+	)
+	(wire
+		(pts
 			(xy 104.14 120.65) (xy 104.14 123.19)
 		)
@@
 	(wire
 		(pts
+			(xy 68.58 171.45) (xy 62.23 171.45)
+		)
+		(stroke
+			(width 0)
+			(type default)
+		)
+	)
+	(wire
+		(pts
 			(xy 156.21 95.25) (xy 156.21 97.79)
 		)
@@
 	(wire
 		(pts
-			(xy 74.93 181.61) (xy 62.23 181.61)
+			(xy 74.93 181.61) (xy 68.58 181.61)
 		)
 		(stroke
@@
 	(wire
 		(pts
+			(xy 100.33 171.45) (xy 100.33 172.72)
+		)
+		(stroke
+			(width 0)
+			(type default)
+		)
+	)
+	(wire
+		(pts
 			(xy 41.91 39.37) (xy 41.91 41.91)
 		)
@@
 	(wire
 		(pts
-			(xy 74.93 171.45) (xy 62.23 171.45)
+			(xy 74.93 171.45) (xy 68.58 171.45)
+		)
+		(stroke
+			(width 0)
+			(type default)
+		)
+	)
+	(wire
+		(pts
+			(xy 100.33 181.61) (xy 100.33 180.34)
 		)
 		(stroke
@@
 	(wire
 		(pts
-			(xy 62.23 181.61) (xy 62.23 182.88)
+			(xy 68.58 181.61) (xy 68.58 182.88)
 		)
 		(stroke
@@
 		(dnp no)
 		(fields_autoplaced yes)
-		(property "Reference" "C44"
+		(property "Reference" "C45"
 			(at 184.15 58.42 90)
 			(effects
@@
 			(project "ThunderHorse"
 				(path "/ac187c6c-fa53-41cc-bce1-6f39a42a92e8/807a5f6f-4255-4cf0-8d90-acd62bb18590/1e531f33-ba68-434b-8668-a85d28098a3f"
-					(reference "C44")
+					(reference "C45")
 					(unit 1)
 				)
@@
 		(dnp no)
 		(fields_autoplaced yes)
-		(property "Reference" "C42"
+		(property "Reference" "C43"
 			(at 144.78 40.6399 0)
 			(effects
@@
 			(project "ThunderHorse"
 				(path "/ac187c6c-fa53-41cc-bce1-6f39a42a92e8/807a5f6f-4255-4cf0-8d90-acd62bb18590/1e531f33-ba68-434b-8668-a85d28098a3f"
-					(reference "C42")
+					(reference "C43")
 					(unit 1)
 				)
@@
 		(dnp no)
 		(fields_autoplaced yes)
-		(property "Reference" "C45"
+		(property "Reference" "C46"
 			(at 184.15 72.39 90)
 			(effects
@@
 			(project "ThunderHorse"
 				(path "/ac187c6c-fa53-41cc-bce1-6f39a42a92e8/807a5f6f-4255-4cf0-8d90-acd62bb18590/1e531f33-ba68-434b-8668-a85d28098a3f"
-					(reference "C45")
+					(reference "C46")
 					(unit 1)
 				)
@@
 	(symbol
 		(lib_id "power:+5V")
-		(at 62.23 170.18 0)
+		(at 68.58 170.18 0)
 		(unit 1)
 		(exclude_from_sim no)
@@
 		(dnp no)
 		(fields_autoplaced yes)
-		(property "Reference" "#PWR072"
-			(at 62.23 173.99 0)
+		(property "Reference" "#PWR074"
+			(at 68.58 173.99 0)
 			(effects
 				(font
@@
 		)
 		(property "Value" "VBAT"
-			(at 62.23 165.1 0)
+			(at 68.58 165.1 0)
 			(effects
 				(font
@@
 		)
 		(property "Footprint" ""
-			(at 62.23 170.18 0)
+			(at 68.58 170.18 0)
 			(effects
 				(font
@@
 		)
 		(property "Datasheet" ""
-			(at 62.23 170.18 0)
+			(at 68.58 170.18 0)
 			(effects
 				(font
@@
 		)
 		(property "Description" "Power symbol creates a global label with name \"+5V\""
-			(at 62.23 170.18 0)
+			(at 68.58 170.18 0)
 			(effects
 				(font
@@
 			(project "ThunderHorse"
 				(path "/ac187c6c-fa53-41cc-bce1-6f39a42a92e8/807a5f6f-4255-4cf0-8d90-acd62bb18590/1e531f33-ba68-434b-8668-a85d28098a3f"
-					(reference "#PWR072")
+					(reference "#PWR074")
 					(unit 1)
 				)
@@
 	(symbol
 		(lib_id "power:GND")
-		(at 62.23 182.88 0)
+		(at 68.58 182.88 0)
 		(unit 1)
 		(exclude_from_sim no)
@@
 		(dnp no)
 		(fields_autoplaced yes)
-		(property "Reference" "#PWR073"
-			(at 62.23 189.23 0)
+		(property "Reference" "#PWR075"
+			(at 68.58 189.23 0)
 			(effects
 				(font
@@
 		)
 		(property "Value" "GND"
-			(at 62.23 187.96 0)
+			(at 68.58 187.96 0)
 			(effects
 				(font
@@
 		)
 		(property "Footprint" ""
-			(at 62.23 182.88 0)
+			(at 68.58 182.88 0)
 			(effects
 				(font
@@
 		)
 		(property "Datasheet" ""
-			(at 62.23 182.88 0)
+			(at 68.58 182.88 0)
 			(effects
 				(font
@@
 		)
 		(property "Description" "Power symbol creates a global label with name \"GND\" , ground"
-			(at 62.23 182.88 0)
+			(at 68.58 182.88 0)
 			(effects
 				(font
@@
 			(project "ThunderHorse"
 				(path "/ac187c6c-fa53-41cc-bce1-6f39a42a92e8/807a5f6f-4255-4cf0-8d90-acd62bb18590/1e531f33-ba68-434b-8668-a85d28098a3f"
-					(reference "#PWR073")
+					(reference "#PWR075")
 					(unit 1)
 				)
@@
 		(on_board yes)
 		(dnp no)
-		(property "Reference" "#PWR074"
+		(property "Reference" "#PWR072"
 			(at 68.58 40.64 0)
 			(effects
@@
 			(project "ThunderHorse"
 				(path "/ac187c6c-fa53-41cc-bce1-6f39a42a92e8/807a5f6f-4255-4cf0-8d90-acd62bb18590/1e531f33-ba68-434b-8668-a85d28098a3f"
-					(reference "#PWR074")
+					(reference "#PWR072")
 					(unit 1)
 				)
@@
 		(dnp no)
 		(fields_autoplaced yes)
-		(property "Reference" "C43"
+		(property "Reference" "C44"
 			(at 184.15 44.45 90)
 			(effects
@@
 			(project "ThunderHorse"
 				(path "/ac187c6c-fa53-41cc-bce1-6f39a42a92e8/807a5f6f-4255-4cf0-8d90-acd62bb18590/1e531f33-ba68-434b-8668-a85d28098a3f"
-					(reference "C43")
+					(reference "C44")
 					(unit 1)
 				)
@@
 			)
 		)
-		(property "Footprint" "Custom_Parts:PAD_3_SQUARE_SOLID_2.0x2.0mm_P2.5mm"
+		(property "Footprint" "Custom_Parts:PAD_3_SQUARE_SOLID_2.5x2.5mm_P4.0mm"
 			(at 187.96 134.62 0)
 			(effects
@@
 		(dnp no)
 		(fields_autoplaced yes)
-		(property "Reference" "#PWR075"
+		(property "Reference" "#PWR073"
 			(at 68.58 104.14 0)
 			(effects
@@
 			(project "ThunderHorse"
 				(path "/ac187c6c-fa53-41cc-bce1-6f39a42a92e8/807a5f6f-4255-4cf0-8d90-acd62bb18590/1e531f33-ba68-434b-8668-a85d28098a3f"
-					(reference "#PWR075")
+					(reference "#PWR073")
 					(unit 1)
 				)
@@
 					(unit 1)
 				)
+			)
+		)
+	)
+	(symbol
+		(lib_id "Device:C")
+		(at 100.33 176.53 0)
+		(unit 1)
+		(exclude_from_sim no)
+		(in_bom yes)
+		(on_board yes)
+		(dnp no)
+		(fields_autoplaced yes)
+		(property "Reference" "C42"
+			(at 104.14 175.2599 0)
+			(effects
+				(font
+					(size 1.27 1.27)
+				)
+				(justify left)
+			)
+		)
+		(property "Value" "10u"
+			(at 104.14 177.7999 0)
+			(effects
+				(font
+					(size 1.27 1.27)
+				)
+				(justify left)
+			)
+		)
+		(property "Footprint" "Capacitor_SMD:C_1206_3216Metric"
+			(at 101.2952 180.34 0)
+			(effects
+				(font
+					(size 1.27 1.27)
+				)
+				(hide yes)
+			)
+		)
+		(property "Datasheet" "~"
+			(at 100.33 176.53 0)
+			(effects
+				(font
+					(size 1.27 1.27)
+				)
+				(hide yes)
+			)
+		)
+		(property "Description" "Unpolarized capacitor"
+			(at 100.33 176.53 0)
+			(effects
+				(font
+					(size 1.27 1.27)
+				)
+				(hide yes)
+			)
+		)
+		(pin "1"
+		)
+		(pin "2"
+		)
+		(instances
+			(project "ThunderHorse"
+				(path "/ac187c6c-fa53-41cc-bce1-6f39a42a92e8/807a5f6f-4255-4cf0-8d90-acd62bb18590/1e531f33-ba68-434b-8668-a85d28098a3f"
+					(reference "C42")
+					(unit 1)
+				)

Commit message: Layout replication
Updated the ESC schematic to allow for layout replication.
Updated the PCB layout.
Changed lines of the file:
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@@
 		(company "DavidMolTor")
+	)
+	(rectangle
+		(start 12.7 12.7)
+		(end 20.32 20.32)
+		(stroke
+			(width 0)
+			(type default)
+		)
+		(fill
+			(type none)
+		)
 	)
 	(text_box "GATE DRIVER"
@@
 			)
 		)
+	)
+	(rule_area
+		(polyline
+			(pts
+				(xy 20.32 20.32) (xy 20.32 193.04) (xy 119.38 193.04) (xy 119.38 158.75) (xy 276.86 158.75) (xy 276.86 20.32)
+			)
+			(stroke
+				(width 0)
+				(type dash)
+			)
+			(fill
+				(type none)
+			)
+		)
+	)
+	(netclass_flag ""
+		(length 2.54)
+		(shape round)
+		(at 22.86 20.32 0)
+		(fields_autoplaced yes)
+		(effects
+			(font
+				(size 1.27 1.27)
+			)
+			(justify left bottom)
+		)
+		(property "Netclass" ""
+			(at -294.64 -59.69 0)
+			(effects
+				(font
+					(size 1.27 1.27)
+				)
+			)
+		)
+		(property "Component Class" "ESC1"
+			(at 23.5585 17.78 0)
+			(effects
+				(font
+					(size 1.27 1.27)
+					(italic yes)
+				)
+				(justify left)
+			)
+		)

Commit message: Initial layout
Completed an initial layout of the main components.

TODO
Route the ESCs and check the result.
Parts:
- renumbered C35 to C36, C36 to C37, C37 to C38, C38 to C39, C39 to C40, C40 to C41, C41 to C42, C42 to C43, C43 to C44, C44 to C45, C45 to C46, C46 to C47, Q2 to Q1, Q3 to Q2, Q4 to Q3, U7 to U8, U8 to U9

Commit message: Settings and ESC layout
Updated the PCB configuration options for manufacturing.
Completed the initial ESC layout.

TODO:
Replicate ESC layout.
Parts:
- J8: footprint Custom_Parts:PAD_3_SQUARE_SOLID_2.5x2.5mm_P4.0mm -> Custom_Parts:PAD_3_SQUARE_SOLID_2.5x2.5mm_P4.0mm_MOTOR
Changed lines of the file:
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@@
 			)
 		)
-		(property "Footprint" "Custom_Parts:PAD_3_SQUARE_SOLID_2.5x2.5mm_P4.0mm"
+		(property "Footprint" "Custom_Parts:PAD_3_SQUARE_SOLID_2.5x2.5mm_P4.0mm_MOTOR"
 			(at 187.96 134.62 0)
 			(effects
