File: Receiver.kicad_sch (KiCad schematic)
At the start: 37 parts, among them SW2 TS2306A, U19 ESP32-C3, U20 AT2401C, U21 TPRT9013-33, U22 SX1280IMLTRT, Y2 40MHz, Y3 52MHz/10ppm

Commit message: Oscillator and IMU layout
Updated the oscillator layout for the RP2350.
Updated the IMU layout for the IMU.
Parts:
- renumbered C98 to C100, C99 to C101, C100 to C102, C101 to C103, C102 to C104, C103 to C105, C104 to C106, C84 to C86, C85 to C87, C86 to C88, C87 to C89, C88 to C90, C89 to C91, C90 to C92, C91 to C93, C92 to C94, C93 to C95, C94 to C96, C95 to C97, C96 to C98, C97 to C99

Commit message: Power layout and regulators
Changed the LDO regulators to TLV767.
Added missing power connections.

TODO:
Start the ELRS module layout.
Review previous iterations.
Parts:
- removed U21: TPRT9013-33, Package_TO_SOT_SMD:SOT-23-5, symbol Regulator_Linear:TLV70233_SOT23-5
- added U3: TLV76733DRVX, Package_SON:WSON-6-1EP_2x2mm_P0.65mm_EP1x1.6mm_ThermalVias, symbol Custom_Parts:TLV76733DRVX
Connections:
- net 3V3_RX: now also U3.1 (OUT), U3.2 (SNS)
- net 5V: now also U3.4 (EN), U3.6 (IN)
- net GND: now also U3.3 (GND), U3.5 (GND), U3.7 (PAD)

Commit message: Voltage detection
Added a VBUS voltage detection for the RP.
Minor layout changes.
Parts:
- renumbered C87 to C100, C91 to C101, C100 to C102, C89 to C104, C92 to C105, C96 to C106, C104 to C86, C105 to C87, C101 to C88, C102 to C89, C86 to C90, C88 to C91, C90 to C92, C97 to C96, C98 to C97, C106 to C98, R89 to R87, R85 to R89, R86 to R90, R87 to R91, U22 to U19, U19 to U20, U3 to U21, U20 to U22, Y3 to Y2, Y2 to Y3
